File: AutoCompost_Placa/AutoCompost_Placa.kicad_sch (KiCad schematic)
At the start: 28 parts, among them U1 LM7805_TO220, U2 ESP32-DEVKIT-V1

Commit message: Agregado de botones
Parts:
- added CrusherButton1, FanButton1, MixerButton1: Molex 0.100, Conectores_Molex:Molex_100_2pines, symbol Conectores_Molex:Molex_100_2pines
Connections:
- net GND: now also QCrusher1.1, QFan1.1, QMixer1.1, CrusherButton1.2, FanButton1.2, MixerButton1.2; no longer QCrusher1.3, QFan1.3, QMixer1.3
- net at SSR_Cruhser1.4 (-): now also QCrusher1.3; no longer QCrusher1.1
- net MixerBtn: now reaches U2.19 (D34)
- net MixerBtn: now also MixerButton1.1
- net CrusherBtn: now reaches U2.20 (D35)
- net CrusherBtn: now also CrusherButton1.1
- net FanBtn: now reaches U2.21 (D32)
- net FanBtn: now also FanButton1.1
- net at SSR_Mixer1.4 (-): now also QMixer1.3; no longer QMixer1.1
- net at SSR_Fan1.4 (-): now also QFan1.3; no longer QFan1.1
Other:
- moved on the sheet: DHT1, DS18B1, HC-SR1, LCD1, Lock1, Lock2, QLock1, R1, R2, RFan1, RLock1, RMixer1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

Commit message: Agregado de esquematico con rele
Parts:
- added R2, R3, R4: 10k, Resistor_THT:R_Axial_DIN0309_L9.0mm_D3.2mm_P12.70mm_Horizontal, symbol Device:R
Connections:
- net 3V3: now also CrusherButton1.1, FanButton1.1, MixerButton1.1
- net CrusherBtn: now also CrusherButton1.2, R3.2; no longer CrusherButton1.1
- net FanBtn: now also FanButton1.2, R4.2; no longer FanButton1.1
- net GND: now also R2.1, R3.1, R4.1; no longer CrusherButton1.2, FanButton1.2, MixerButton1.2
- net MixerBtn: now also MixerButton1.2, R2.2; no longer MixerButton1.1
