File: Placa_Rele/Placa_Rele/_autosave-Placa_Rele.kicad_pcb (KiCad board)
At the start: 2 copper layers, 43 parts, among them J1 Screw_Terminal_Crusher1, J2 MixerScrewTerminal1, J3 FanScrewTerminal1, K1 FINDER-36.11, K2 FINDER-36.11, K3 FINDER-36.11, Q1 2N3904, Q2 2N3904, Q3 2N3904, U1 LM7805_TO220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

Commit message: Primero Version de PCB con PCB_rele
Primer PCB terminado, los componentes no estan en su posicion final.
El principal problema fue la conexion de 5V, 3v3 y GND en los conectores
del ultrasonico, LCD y DHT.
Parts:
- moved MixerButton1 286.8 mm to (99.1, 84.5), turned to 90 degrees
- moved LCD1 282.3 mm to (100.3, 122.2), turned to 180 degrees
- moved HC-SR1 282.0 mm to (100.3, 112.0), turned to 180 degrees
- moved Vext1 270.5 mm to (99.6, 68.6), turned to 90 degrees
- moved C1 265.0 mm to (113.1, 72.3), turned to 180 degrees
- moved FanButton1 264.5 mm to (99.2, 92.0), turned to 90 degrees
- moved CrusherButton1 257.8 mm to (99.1, 77.5), turned to 90 degrees
- moved R1 246.4 mm to (108.0, 129.5)
- moved C2 235.9 mm to (144.6, 68.5)
- moved R2 232.3 mm to (111.8, 97.8), turned to -90 degrees
- moved R4 230.5 mm to (109.2, 80.0), turned to -90 degrees
- moved DHT1 228.6 mm to (99.0, 131.2), turned to -90 degrees
- moved DS18B1 226.0 mm to (98.9, 101.9), turned to 90 degrees
- moved R3 226.0 mm to (114.3, 80.0), turned to -90 degrees
- moved R5 220.0 mm to (119.9, 86.3), turned to -90 degrees
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Connections:
- U2 pad 15: unconnected-(U2-D23-Pad15) -> /DHT
- U2 pad 19: /MixerBtn -> /Crusher
- U2 pad 20: /CrusherBtn -> /Mixer
- U2 pad 21: /FanBtn -> /Fan
- U2 pad 25: /DHT -> unconnected-(U2-D27-Pad25)
- U2 pad 3: /Crusher -> /CrusherBtn
- U2 pad 4: /Mixer -> /MixerBtn
- U2 pad 5: /Fan -> /FanBtn
Routing:
- net GND: track 55.3 -> 487.8 mm
- net 5V: track 61.8 -> 315.2 mm
- net /3V3: track 0.00 -> 154.4 mm
- net /VCC: track 0.00 -> 79.4 mm
- net /CrusherBtn: track 0.00 -> 38.1 mm
- net /Lock: track 0.00 -> 37.0 mm
- net /DHT: track 0.00 -> 34.2 mm
- net /DS18B20: track 0.00 -> 34.0 mm
- net /MixerBtn: track 0.00 -> 33.3 mm
- net /FanBtn: track 0.00 -> 32.4 mm
- net /Lid: track 0.00 -> 32.1 mm
- net /Echo_HC-SR04: track 0.00 -> 31.7 mm
- net /LCD_SDA: track 0.00 -> 28.7 mm
- net /Trig_HC-SR04: track 0.00 -> 28.2 mm
- net /LCD_SCL: track 0.00 -> 23.0 mm
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