File: Placa_Rele/Placa_Rele/Placa_Rele.kicad_pcb (KiCad board)
At the start: 2 copper layers, 43 parts, among them J1 Screw_Terminal_Crusher1, J2 MixerScrewTerminal1, J3 FanScrewTerminal1, K1 FINDER-36.11, K2 FINDER-36.11, K3 FINDER-36.11, Q1 2N3904, Q2 2N3904, Q3 2N3904, U1 LM7805_TO220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

Commit message: Modificacion de PCB
Se cambiaron los ordenes de los GPIO asi DHT y DS18B estaban en los
primeros GPIOS y facilitaba el ruteo.
Parts:
- moved MixerButton1 287.1 mm to (99.1, 110.5), turned to 90 degrees
- moved HC-SR1 283.4 mm to (100.3, 121.9), turned to 180 degrees
- moved Vext1 270.5 mm to (99.6, 68.6), turned to 90 degrees
- moved LCD1 267.1 mm to (115.6, 121.9), turned to 180 degrees
- moved C1 265.0 mm to (113.1, 72.3), turned to 180 degrees
- moved FanButton1 264.6 mm to (99.2, 104.1), turned to 90 degrees
- moved CrusherButton1 257.2 mm to (99.1, 97.8), turned to 90 degrees
- moved C2 235.9 mm to (144.6, 68.5)
- moved DHT1 226.6 mm to (99.1, 78.7), turned to -90 degrees
- moved DS18B1 226.5 mm to (99.0, 88.2), turned to 90 degrees
- moved R3 225.2 mm to (120.7, 109.2), turned to 180 degrees
- moved R2 222.5 mm to (120.0, 88.9), turned to 180 degrees
- moved R1 222.4 mm to (120.0, 83.8), turned to 180 degrees
- moved R5 222.0 mm to (120.7, 104.1), turned to 180 degrees
- moved R4 221.9 mm to (120.7, 99.1), turned to 180 degrees
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Connections:
- U2 pad 19: /MixerBtn -> /Crusher
- U2 pad 20: /CrusherBtn -> /Mixer
- U2 pad 21: /FanBtn -> /Fan
- U2 pad 25: /DHT -> unconnected-(U2-D27-Pad25)
- U2 pad 3: /Crusher -> /DHT
- U2 pad 4: /Mixer -> /DS18B20
- U2 pad 5: /Fan -> /CrusherBtn
- U2 pad 7: unconnected-(U2-TX2-Pad7) -> /FanBtn
- U2 pad 8: /DS18B20 -> /MixerBtn
Routing:
- net GND: track 55.3 -> 497.2 mm
- net 5V: track 61.8 -> 285.3 mm
- net /3V3: track 0.00 -> 81.5 mm
- net /VCC: track 0.00 -> 79.4 mm
- net /Lock: track 0.00 -> 37.0 mm
- net /DHT: track 0.00 -> 34.3 mm
- net /Echo_HC-SR04: track 0.00 -> 33.2 mm
- net /Lid: track 0.00 -> 32.1 mm
- net /DS18B20: track 0.00 -> 31.5 mm
- net /MixerBtn: track 0.00 -> 30.0 mm
- net /FanBtn: track 0.00 -> 29.6 mm
- net /Trig_HC-SR04: track 0.00 -> 29.6 mm
- net /CrusherBtn: track 0.00 -> 29.4 mm
- net Net-(QLock1-B): track 0.00 -> 18.9 mm
- net /Fan: track 31.7 -> 13.9 mm
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
Commit message: Placa final con  reles pero sin LEDS
Parts:
- removed 5V1: Molex 0.156, Conectores_Molex:Molex_156_2pines
- moved Lock2 30.5 mm to (199.4, 68.6)
- moved C2 28.2 mm to (172.7, 68.6), turned to 180 degrees
- moved QLock1 10.1 mm to (185.4, 68.6)
- moved RLock1 9.92 mm to (177.8, 76.2)
- moved R13 8.87 mm to (168.9, 81.2)
- moved D1 8.54 mm to (182.9, 123.1)
- moved D2 8.54 mm to (182.9, 104.2)
- moved D3 8.54 mm to (182.9, 85.2)
- moved J1 8.54 mm to (215.9, 123.3)
- moved J2 8.54 mm to (215.9, 104.3)
- moved K1 8.54 mm to (190.1, 126.8)
- moved K2 8.54 mm to (190.1, 107.8)
- moved R10 8.54 mm to (167.6, 100.3)
- moved R11 8.54 mm to (162.6, 113.0)
- moved R14 8.54 mm to (162.6, 94.1)
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Routing:
- net GND: track 497.2 -> 537.6 mm
- net /VCC: track 79.4 -> 107.0 mm
- net 5V: track 285.3 -> 307.7 mm
- net Net-(QLock1-C): track 9.78 -> 19.9 mm
- net Net-(QLock1-B): track 18.9 -> 10.8 mm
- net /Fan: track 13.9 -> 21.8 mm
- net /Lid: track 32.1 -> 38.7 mm
- net /LCD_SDA: track 13.3 -> 19.4 mm
- net /3V3: track 81.5 -> 87.0 mm
- net /LCD_SCL: track 8.01 -> 12.7 mm
- net /Crusher: track 15.4 -> 11.3 mm
- net /Trig_HC-SR04: track 29.6 -> 32.1 mm
- net /Mixer: track 13.1 -> 10.7 mm
- net /Lock: track 37.0 -> 38.3 mm
- net /Echo_HC-SR04: track 33.2 -> 32.1 mm
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
Commit message: Placa de potencia terminada con borneras
Other:
- board outline added: 132.1 x 78.7 mm

Commit message: feat: Agregado de placa para pcbway
Parts:
- added LEDs1: Molex 0.100, Conectores_Molex:Molex_100_4pines, F.Cu at (78.7, 53.3)
- moved Q1 90.7 mm to (96.4, 86.5)
- moved Q2 90.7 mm to (96.4, 66.2)
- moved RLock1 90.7 mm to (100.3, 29.2)
- moved U3 90.7 mm to (96.4, 80.2)
- moved U4 90.7 mm to (96.4, 61.1)
- moved U5 90.7 mm to (96.4, 42.0)
- moved C1 90.7 mm to (33.1, 19.6)
- moved C2 90.7 mm to (95.2, 21.6)
- moved CrusherButton1 90.7 mm to (21.5, 50.8)
- moved D1 90.7 mm to (105.3, 76.2)
- moved D2 90.7 mm to (105.3, 57.2)
- moved D3 90.7 mm to (105.3, 38.2)
- moved DHT1 90.7 mm to (21.5, 31.8)
- moved DS18B1 90.7 mm to (21.4, 41.2)
- moved FanButton1 90.7 mm to (21.6, 57.1)
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Connections:
- U2 pad 23: unconnected-(U2-D25-Pad23) -> /Lid
- U2 pad 24: /Lid -> /Led1
- U2 pad 25: unconnected-(U2-D27-Pad25) -> /Led2
- U2 pad 26: unconnected-(U2-D14-Pad26) -> /Led3
- U2 pad 27: unconnected-(U2-D12-Pad27) -> /Led4
Routing:
- net /Lid: track 38.7 -> 43.8 mm
- net /Led4: track 0.00 -> 3.81 mm
- net /Led3: track 0.00 -> 3.81 mm
- net /Led2: track 0.00 -> 3.81 mm
- net /Led1: track 0.00 -> 3.81 mm
- net /Fan: track 21.8 -> 25.3 mm
- net /Lock: track 38.3 -> 41.4 mm
